Commit message: fixed transforms and got slam working

File: src/rc_car_description/urdf/rc_car.urdf.xacro (robot description, xacro)
@@ -292,5 +292,5 @@
     <inertial>
       <origin xyz="0 0 0" rpy="0 0 0"/>
-      <mass value="0.83"/>
+      <mass value="0.15"/>
       <inertia ixx="0.000830" ixy="0" ixz="0"
                iyy="0.000830" iyz="0"

Commit message: urdf depth camera updates

File: src/rc_car_description/urdf/rc_car.urdf.xacro (robot description, xacro)
@@ -360,5 +360,5 @@
     <origin xyz="${chassis_length*0.45} 0 ${chassis_height*0.8}" rpy="0 0 0"/>
   </joint>
-  <!-- <link name="depth_camera_optical_link">
+  <link name="depth_camera_optical_link">
     <xacro:dummy_inertia/>
   </link>
@@ -367,4 +367,4 @@
     <child  link="depth_camera_optical_link"/>
     <origin xyz="0 0 0" rpy="${-pi/2} 0 ${-pi/2}"/>
-  </joint> -->
+  </joint>
 </robot>
