Commit message: added 2d lidar and slamtoolbox. map getting messed up because of issues with odom -> basefootprint transform

File: src/rc_car_description/urdf/ignition_plugins.xacro (robot description, xacro)
@@ -143,46 +143,30 @@
   </gazebo>
   <!-- ============================================================
-       3D LIDAR SENSOR  (Velodyne VLP-16 style)
-       16 channels, 360 deg horizontal, 100m range
+       2D LIDAR SENSOR (planar scan)
+       Simulates a single-layer laser scanner for Nav2/SLAM
        Note: no XML comments inside sensor block — Gazebo 6 parser bug
   ============================================================ -->
-  <gazebo reference="lidar_link">
-    <sensor name="lidar_3d" type="gpu_lidar">
-    <!-- <sensor name="lidar_3d" type="lidar"> -->
-      <always_on>true</always_on>
+ <gazebo reference="lidar_link">
+    <sensor name="laser_2d" type="gpu_lidar"> <!-- Changed from ray to gpu_lidar -->
+      <gz_frame_id>lidar_link</gz_frame_id> <!-- Required for correct TF in ROS -->
       <update_rate>10</update_rate>
-      <visualize>true</visualize>
-      <topic>/lidar</topic>
-      <!-- <plugin filename="libignition-gazebo-sensors-system.so"
-              name="ignition::gazebo::systems::Sensors">
-      </plugin> -->
+      <topic>scan</topic>
       <lidar>
         <scan>
           <horizontal>
-            <samples>1800</samples>
+            <samples>360</samples>
             <resolution>1</resolution>
-            <min_angle>-3.14159265</min_angle>
-            <max_angle>3.14159265</max_angle>
+            <min_angle>-3.14159</min_angle>
+            <max_angle>3.14159</max_angle>
           </horizontal>
-          <vertical>
-            <samples>16</samples>
-            <resolution>1</resolution>
-            <min_angle>-0.261799</min_angle>
-            <max_angle>0.261799</max_angle>
-          </vertical>
         </scan>
         <range>
-          <min>0.10</min>
-          <max>100.0</max>
+          <min>0.1</min>
+          <max>30.0</max>
           <resolution>0.01</resolution>
         </range>
-        <noise>
-          <type>gaussian</type>
-          <mean>0.0</mean>
-          <stddev>0.01</stddev>
-        </noise>
       </lidar>
+      <visualize>true</visualize>
     </sensor>
-    <material>Gazebo/DarkGrey</material>
   </gazebo>
   <!-- ============================================================

Commit message: got depth camera working in sim

File: src/rc_car_description/urdf/ignition_plugins.xacro (robot description, xacro)
@@ -1,5 +1,4 @@
 <?xml version="1.0"?>
 <robot xmlns:xacro="http://www.ros.org/wiki/xacro">
-  <!-- Ignition Gazebo 6 (Fortress) plugin configuration -->
   <!-- ============================================================
        WHEEL CONTACT PROPERTIES
@@ -99,5 +98,4 @@
   <!-- ============================================================
        ROS2 CONTROL — Ignition Gazebo 6 plugin
-       Uses ign_ros2_control (Humble compatible)
   ============================================================ -->
   <gazebo>
@@ -118,5 +116,4 @@
   <!-- ============================================================
        IMU SENSOR
-       Note: no XML comments inside sensor block — Gazebo 6 parser bug
   ============================================================ -->
   <gazebo reference="imu_link">
@@ -143,11 +140,9 @@
   </gazebo>
   <!-- ============================================================
-       2D LIDAR SENSOR (planar scan)
-       Simulates a single-layer laser scanner for Nav2/SLAM
-       Note: no XML comments inside sensor block — Gazebo 6 parser bug
+       2D LIDAR SENSOR
   ============================================================ -->
  <gazebo reference="lidar_link">
-    <sensor name="laser_2d" type="gpu_lidar"> <!-- Changed from ray to gpu_lidar -->
-      <gz_frame_id>lidar_link</gz_frame_id> <!-- Required for correct TF in ROS -->
+    <sensor name="laser_2d" type="gpu_lidar">
+      <gz_frame_id>lidar_link</gz_frame_id>
       <update_rate>10</update_rate>
       <topic>scan</topic>
@@ -171,6 +166,5 @@
   </gazebo>
   <!-- ============================================================
-       FRONT CAMERA SENSOR
-       Note: no XML comments inside sensor block — Gazebo 6 parser bug
+       FRONT CAMERA
   ============================================================ -->
   <gazebo reference="camera_link">
@@ -178,9 +172,6 @@
       <always_on>true</always_on>
       <update_rate>30</update_rate>
-      <visualize>false</visualize>
+      <visualize>true</visualize>
       <topic>/camera/image_raw</topic>
-      <!-- <plugin filename="libignition-gazebo-sensors-system.so"
-              name="ignition::gazebo::systems::Sensors">
-      </plugin> -->
       <camera>
         <horizontal_fov>1.047</horizontal_fov>
@@ -202,3 +193,34 @@
     </sensor>
   </gazebo>
+  <!-- ============================================================
+       DEPTH CAMERA
+  ============================================================ -->
+  <gazebo reference="depth_camera_link">
+    <sensor name="depth_camera" type="depth_camera">
+      <always_on>true</always_on>
+      <update_rate>30</update_rate>
+      <visualize>true</visualize>
+      <min_depth>0.1</min_depth>
+      <max_depth>100.0</max_depth>
+      <gz_frame_id>depth_camera_link</gz_frame_id>
+      <topic>/depth_camera/depth_image</topic>
+      <camera>
+        <horizontal_fov>1.047</horizontal_fov>
+        <image>
+          <width>640</width>
+          <height>480</height>
+          <format>R_FLOAT32</format>
+        </image>
+        <clip>
+          <near>0.1</near>
+          <far>15.0</far>
+        </clip>
+        <!-- <noise>
+          <type>gaussian</type>
+          <mean>0.0</mean>
+          <stddev>0.007</stddev>
+        </noise> -->
+      </camera>
+    </sensor>
+  </gazebo>
 </robot>

File: src/rc_car_description/urdf/rc_car.urdf.xacro (robot description, xacro)
@@ -340,3 +340,31 @@
     <origin xyz="0 0 0" rpy="${-pi/2} 0 ${-pi/2}"/>
   </joint>
+  <!-- ============================================================
+       DEPTH CAMERA LINKS
+  ============================================================ -->
+  <link name="depth_camera_link">
+    <xacro:dummy_inertia/>
+    <visual>
+      <origin xyz="0 0 0" rpy="0 0 0"/>
+      <geometry><box size="0.02 0.04 0.02"/></geometry>
+      <material name="dark_grey"/>
+    </visual>
+    <collision>
+      <origin xyz="0 0 0" rpy="0 0 0"/>
+      <geometry><box size="0.02 0.04 0.02"/></geometry>
+    </collision>
+  </link>
+  <joint name="depth_camera_joint" type="fixed">
+    <parent link="base_link"/>
+    <child  link="depth_camera_link"/>
+    <origin xyz="${chassis_length*0.45} 0 ${chassis_height*0.8}" rpy="0 0 0"/>
+  </joint>
+  <!-- <link name="depth_camera_optical_link">
+    <xacro:dummy_inertia/>
+  </link>
+  <joint name="depth_camera_optical_joint" type="fixed">
+    <parent link="depth_camera_link"/>
+    <child  link="depth_camera_optical_link"/>
+    <origin xyz="0 0 0" rpy="${-pi/2} 0 ${-pi/2}"/>
+  </joint> -->
 </robot>

Commit message: trying to get gazebo physics working properly

File: src/rc_car_description/urdf/ignition_plugins.xacro (robot description, xacro)
@@ -9,15 +9,15 @@
           <friction>
             <ode>
-              <mu>100.0</mu>
-              <mu2>100.0</mu2>
-              <fdir1>1 0 0</fdir1>
-              <slip1>0.0</slip1>
-              <slip2>0.0</slip2>
-            </ode>
-          </friction>
-          <contact>
-            <ode>
-              <kp>1000000.0</kp>
-              <kd>1.0</kd>
+              <mu>1.0</mu>
+              <mu2>1.2</mu2>
+              <fdir1>1 0 0</fdir1>
+              <slip1>0.01</slip1>
+              <slip2>0.02</slip2>
+            </ode>
+          </friction>
+          <contact>
+            <ode>
+              <kp>1.0e5</kp>
+              <kd>10.0</kd>
               <min_depth>0.001</min_depth>
             </ode>
@@ -32,15 +32,15 @@
           <friction>
             <ode>
-              <mu>100.0</mu>
-              <mu2>100.0</mu2>
-              <fdir1>1 0 0</fdir1>
-              <slip1>0.0</slip1>
-              <slip2>0.0</slip2>
-            </ode>
-          </friction>
-          <contact>
-            <ode>
-              <kp>1000000.0</kp>
-              <kd>1.0</kd>
+              <mu>1.0</mu>
+              <mu2>1.2</mu2>
+              <fdir1>1 0 0</fdir1>
+              <slip1>0.01</slip1>
+              <slip2>0.02</slip2>
+            </ode>
+          </friction>
+          <contact>
+            <ode>
+              <kp>1.0e5</kp>
+              <kd>10.0</kd>
               <min_depth>0.001</min_depth>
             </ode>
@@ -55,15 +55,15 @@
           <friction>
             <ode>
-              <mu>100.0</mu>
-              <mu2>100.0</mu2>
-              <fdir1>1 0 0</fdir1>
-              <slip1>0.0</slip1>
-              <slip2>0.0</slip2>
-            </ode>
-          </friction>
-          <contact>
-            <ode>
-              <kp>1000000.0</kp>
-              <kd>1.0</kd>
+              <mu>1.0</mu>
+              <mu2>1.2</mu2>
+              <fdir1>1 0 0</fdir1>
+              <slip1>0.01</slip1>
+              <slip2>0.02</slip2>
+            </ode>
+          </friction>
+          <contact>
+            <ode>
+              <kp>1.0e5</kp>
+              <kd>10.0</kd>
               <min_depth>0.001</min_depth>
             </ode>
@@ -78,15 +78,15 @@
           <friction>
             <ode>
-              <mu>100.0</mu>
-              <mu2>100.0</mu2>
-              <fdir1>1 0 0</fdir1>
-              <slip1>0.0</slip1>
-              <slip2>0.0</slip2>
-            </ode>
-          </friction>
-          <contact>
-            <ode>
-              <kp>1000000.0</kp>
-              <kd>1.0</kd>
+              <mu>1.0</mu>
+              <mu2>1.2</mu2>
+              <fdir1>1 0 0</fdir1>
+              <slip1>0.01</slip1>
+              <slip2>0.02</slip2>
+            </ode>
+          </friction>
+          <contact>
+            <ode>
+              <kp>1.0e5</kp>
+              <kd>10.0</kd>
               <min_depth>0.001</min_depth>
             </ode>

File: src/rc_car_description/urdf/rc_car.ros2_control.xacro (robot description, xacro)
@@ -6,5 +6,11 @@
             </hardware>
             <joint name="front_left_steer_joint">
-                <command_interface name="position"/>
+                <command_interface name="position">
+                    <param name="min">-0.75</param>
+                    <param name="max">0.75</param>
+                    <param name="p">200.0</param>
+                    <param name="i">10.0</param>
+                    <param name="d">5.0</param>
+                </command_interface>
                 <state_interface name="velocity"/>
                 <state_interface name="position">
@@ -12,5 +18,11 @@
             </joint>
             <joint name="front_right_steer_joint">
-                <command_interface name="position"/>
+                <command_interface name="position">
+                    <param name="min">-0.75</param>
+                    <param name="max">0.75</param>
+                    <param name="p">200.0</param>
+                    <param name="i">10.0</param>
+                    <param name="d">5.0</param>
+                </command_interface>
                 <state_interface name="velocity"/>
                 <state_interface name="position">

File: src/rc_car_description/urdf/rc_car.urdf.xacro (robot description, xacro)
@@ -15,12 +15,12 @@
   <xacro:property name="chassis_width"    value="0.20"/>
   <xacro:property name="chassis_height"   value="0.08"/>
-  <xacro:property name="chassis_mass"     value="1.0"/>
+  <xacro:property name="chassis_mass"     value="3.0"/>
   <xacro:property name="wheel_radius"     value="0.055"/>
   <xacro:property name="wheel_width"      value="0.04"/>
-  <xacro:property name="wheel_mass"       value="0.20"/>
+  <xacro:property name="wheel_mass"       value="0.1"/>
   <xacro:property name="wheelbase"        value="0.26"/>
   <xacro:property name="track_width"      value="0.22"/>
   <xacro:property name="ground_clearance" value="0.055"/>
-  <xacro:property name="max_steer"        value="0.6"/>
+  <xacro:property name="max_steer"        value="0.75"/>
   <xacro:property name="hub_size"         value="0.02"/>
   <xacro:property name="hub_mass"         value="0.05"/>
@@ -75,5 +75,5 @@
   <link name="base_link">
     <inertial>
-      <origin xyz="0 0 ${chassis_height/2}" rpy="0 0 0"/>
+      <origin xyz="0 0 0" rpy="0 0 0"/>
       <mass value="${chassis_mass}"/>
       <inertia
@@ -86,5 +86,5 @@
     <visual>
       <origin xyz="0 0 ${chassis_height/2}" rpy="0 0 0"/>
-      <geometry><box size="${chassis_length} ${chassis_width} ${chassis_height}"/></geometry>
+      <geometry><box size="${chassis_length} 0.1 ${chassis_height}"/></geometry>
       <material name="blue"/>
     </visual>
@@ -143,6 +143,6 @@
     <origin xyz="${front_x} ${axle_y} ${axle_z}" rpy="0 0 0"/>
     <axis xyz="0 0 1"/>
-    <limit lower="${-max_steer}" upper="${max_steer}" effort="10.0" velocity="5.0"/>
-    <dynamics damping="0.5" friction="0.1"/>
+    <limit lower="${-max_steer}" upper="${max_steer}" effort="50.0" velocity="5.0"/>
+    <dynamics damping="0.01" friction="0.0"/>
   </joint>
   <link name="front_right_steer_link">
@@ -169,6 +169,6 @@
     <origin xyz="${front_x} ${-axle_y} ${axle_z}" rpy="0 0 0"/>
     <axis xyz="0 0 1"/>
-    <limit lower="${-max_steer}" upper="${max_steer}" effort="10.0" velocity="5.0"/>
-    <dynamics damping="0.5" friction="0.1"/>
+    <limit lower="${-max_steer}" upper="${max_steer}" effort="50.0" velocity="5.0"/>
+    <dynamics damping="0.01" friction="0.0"/>
   </joint>
   <!-- ============================================================
@@ -234,7 +234,7 @@
     <parent link="base_link"/>
     <child  link="rear_left_wheel_link"/>
-    <origin xyz="${rear_x} ${axle_y+wheel_width/2} ${axle_z}" rpy="0 0 0"/>
+    <origin xyz="${rear_x} ${axle_y + hub_size/2 + wheel_width/2} ${axle_z}" rpy="0 0 0"/>
     <axis xyz="0 1 0"/>
-    <dynamics damping="0.01" friction="0.1"/>
+    <dynamics damping="0.0" friction="0.0"/>
   </joint>
   <link name="rear_right_wheel_link">
@@ -262,7 +262,7 @@
     <parent link="base_link"/>
     <child  link="rear_right_wheel_link"/>
-    <origin xyz="${rear_x} ${-(axle_y+wheel_width/2)} ${axle_z}" rpy="0 0 0"/>
+    <origin xyz="${rear_x} ${-(axle_y + hub_size/2 + wheel_width/2)} ${axle_z}" rpy="0 0 0"/>
     <axis xyz="0 1 0"/>
-    <dynamics damping="0.01" friction="0.1"/>
+    <dynamics damping="0.0" friction="0.0"/>
   </joint>
   <!-- ============================================================
